Commit message: Correccion de la direccion de  giro de las articulaciones en el URDF

File: public/urdf/CRS_A465.urdf (robot description, URDF)
Before this commit: robot CRS_A465, 7 links, 6 joints
Links:
- link eslabon_1: geometry collision mesh filename=package://CRS_A465_ok_ok/meshes/eslabon_1.STL; visual mesh filename=package://CRS_A465_ok_ok/meshes/eslabon_1.STL
- link eslabon_2: geometry collision mesh filename=package://CRS_A465_ok_ok/meshes/eslabon_2.STL; visual mesh filename=package://CRS_A465_ok_ok/meshes/eslabon_2.STL
- link eslabon_3: geometry collision mesh filename=package://CRS_A465_ok_ok/meshes/eslabon_3.STL; visual mesh filename=package://CRS_A465_ok_ok/meshes/eslabon_3.STL
- link eslabon_4: geometry collision mesh filename=package://CRS_A465_ok_ok/meshes/eslabon_4.STL; visual mesh filename=package://CRS_A465_ok_ok/meshes/eslabon_4.STL
- link eslabon_5: geometry collision mesh filename=package://CRS_A465_ok_ok/meshes/eslabon_5.STL; visual mesh filename=package://CRS_A465_ok_ok/meshes/eslabon_5.STL
- link eslabon_6: geometry collision mesh filename=package://CRS_A465_ok_ok/meshes/eslabon_6.STL; visual mesh filename=package://CRS_A465_ok_ok/meshes/eslabon_6.STL
- link eslabon_base: geometry collision mesh filename=package://CRS_A465_ok_ok/meshes/eslabon_base.STL; visual mesh filename=package://CRS_A465_ok_ok/meshes/eslabon_base.STL
Joints:
- joint junta_1_2: origin xyz=0 0.33 -8E-05 rpy=0 0 0 -> xyz=0 0.330000000000001 -7.99999999999274E-05 rpy=0 0 0
- joint junta_2_3: axis 0 0 1 -> 0 0 -1; origin xyz=0 0.305 0.000100000000000017 rpy=0 0 0 -> xyz=0 0.305 0.0001 rpy=0 0 0
- joint junta_4_5: axis 0 0 1 -> 0 0 -1

Commit message: Add cast carbon steel texture and shader configuration
- Introduced a new texture file for cast carbon steel.
- Configured shader properties including color, bump mapping, and reflectivity.
- Set parameters for surface finish, including diffuse and specular factors.
- Enabled double-sided rendering and blurry reflections for enhanced visual quality.

File: public/urdf/CRS_A465.urdf (robot description, URDF)
Before this commit: robot CRS_A465, 7 links, 6 joints
Links:
- link eslabon_1: geometry collision mesh filename=package://CRSA465/meshes/eslabon_1.STL; visual mesh filename=package://CRSA465/meshes/eslabon_1.STL
- link eslabon_2: geometry collision mesh filename=package://CRSA465/meshes/eslabon_2.STL; visual mesh filename=package://CRSA465/meshes/eslabon_2.STL
- link eslabon_3: geometry collision mesh filename=package://CRSA465/meshes/eslabon_3.STL; visual mesh filename=package://CRSA465/meshes/eslabon_3.STL
- link eslabon_4: geometry collision mesh filename=package://CRSA465/meshes/eslabon_4.STL; visual mesh filename=package://CRSA465/meshes/eslabon_4.STL
- link eslabon_5: geometry collision mesh filename=package://CRSA465/meshes/eslabon_5.STL; visual mesh filename=package://CRSA465/meshes/eslabon_5.STL
- link eslabon_6: geometry collision mesh filename=package://CRSA465/meshes/eslabon_6.STL; visual mesh filename=package://CRSA465/meshes/eslabon_6.STL
- link eslabon_base: geometry collision mesh filename=package://CRSA465/meshes/eslabon_base.STL; visual mesh filename=package://CRSA465/meshes/eslabon_base.STL

Commit message: Fix: Correction of URDF

File: public/urdf/CRS_A465.urdf (robot description, URDF)
Before this commit: robot CRS_A465, 7 links, 6 joints
Joints:
- joint junta_2_3: axis 0 -1 0 -> 0 1 0
- joint junta_4_5: axis 0 -1 0 -> 0 1 0
