Commit message: Refactor code structure and implemented joint position listener

File: public/urdf/CRSA465.urdf (robot description, URDF)
Before this commit: robot CRS A465 v1 URDF and meshes, 7 links, 6 joints
Joints:
- joint Joint5: parent base_link -> joint4
- joint Joint6: parent base_link -> Joint5
- joint joint2: parent base_link -> joint1
- joint joint3: parent base_link -> joint2
- joint joint4: parent base_link -> joint3

Commit message: fix: update mesh file paths in URDF and adjust camera and lighting settings in RobotArmComponent

File: public/urdf/CRSA465.urdf (robot description, URDF)
Before this commit: robot CRS A465 v1 URDF and meshes, 7 links, 6 joints
Links:
- link Joint5: geometry collision mesh filename=../CRSA465/meshes/Joint5.STL; visual mesh filename=../CRSA465/meshes/Joint5.STL
- link Joint6: geometry collision mesh filename=../CRSA465/meshes/Joint6.STL; visual mesh filename=../CRSA465/meshes/Joint6.STL
- link base_link: geometry collision mesh filename=../CRSA465/meshes/base_link.STL; visual mesh filename=../CRSA465/meshes/base_link.STL
- link joint1: geometry collision mesh filename=../CRSA465/meshes/joint1.STL; visual mesh filename=../CRSA465/meshes/joint1.STL
- link joint2: geometry collision mesh filename=../CRSA465/meshes/joint2.STL; visual mesh filename=../CRSA465/meshes/joint2.STL
- link joint3: geometry collision mesh filename=../CRSA465/meshes/joint3.STL; visual mesh filename=../CRSA465/meshes/joint3.STL
- link joint4: geometry collision mesh filename=../CRSA465/meshes/joint4.STL; visual mesh filename=../CRSA465/meshes/joint4.STL

Commit message: feat(robot-display): add TCP pose display and update styles
- Added a new section in the robot display component to show the TCP pose (position and orientation).
- Updated styles for the pose display to enhance visibility and responsiveness.
- Modified the robot display component to calculate and display the end effector pose.
- Enhanced the robot state service to include position and orientation signals.
- Updated ROS service to handle trajectory planning and CRUD operations for trajectories.
- Added new Python scripts for MoveIt control and position goal handling.
- Included detailed instructions for setting up the ROS2 environment and configuring the robot model.

File: public/urdf/CRSA465.urdf (robot description, URDF)
Before this commit: robot CRSA465, 7 links, 6 joints
Links:
- added link ee_link
- link eslabon_base: mass 5.3549 -> None
Joints:
- added joint junta_ee: type fixed, parent eslabon_6, child ee_link, origin xyz=0 0 0.05 rpy=0 0 0
